File: frontend.kicad_sch (KiCad schematic)
At the start: 20 parts, among them U1 ADG1408YRUZ, U2 ADG1408YRUZ

Commit message: can transceiver; power; mcu
Other:
- note added: "1k sized by FAULT protection, so mishap can't destroy muxes"
- note added: "Cell Voltage Frontend"
- note added: "cell 6 sits 21-25V above ground, and its voltage is a 2.5V - 4.2V difference on that. This circuit removes common-mode voltage mechanically rather than cancelling it. ==> differential sensing We cannot put 21.6V on a 3.3V pin which destroys the pin. And we cannot measure the two ends separately and subtract, because we'd be finding a 3.6V answer by subtracting two ~20V readings, and all the error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"
- moved on the sheet: C1, C2, C3, C4, C5, C6, D1, R1, R15, R16, R2, R3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
