File: power.kicad_sch (KiCad schematic)
At the start: 0 parts

Commit message: can transceiver; power; mcu
Parts:
- added C41, C42, C50: 10uF, symbol Device:C
- added C43, C51: 100nF, symbol Device:C
- added C44: 22uF, symbol Device:C
- added C45, C48, C49: 1uF, symbol Device:C
- added C46: 470pF, symbol Device:C
- added C47: 2.2uF, symbol Device:C
- added D10, D12: D, symbol Device:D
- added D11: SMAJ16A, Diode_SMD:D_SMA, symbol Diode:SMAJ16A
- added F1: PTC 500mA, symbol Device:Fuse
- added FB1: FerriteBead, symbol Device:FerriteBead
- added J4: POWER_IN, symbol Connector:Conn_01x02_Socket
- added L1, L2: L, symbol Device:L
- added Q9: AO3401A, Package_TO_SOT_SMD:SOT-23, symbol Transistor_FET:AO3401A
- added R75, R77, R79: 10k, symbol Device:R
- added R76: 52.3k, symbol Device:R
- added R78: 215k, symbol Device:R
- added R80: 0, symbol Device:R
- added U20: AP63203WU, Package_TO_SOT_SMD:TSOT-23-6, symbol Regulator_Switching:AP63203WU
- added U21: MIC5219-3.3YM5, Package_TO_SOT_SMD:SOT-23-5, symbol Regulator_Linear:MIC5219-3.3YM5
- added U22: TPS61040DBV, Package_TO_SOT_SMD:SOT-23-5, symbol Regulator_Switching:TPS61040DBV
Connections:
- new net: C46.1, U21.4 (BP)
- new net: F1.1, J4.1 (Pin_1)
- new net: R78.2, R79.1, U22.3 (FB)
- new net: L2.1, U22.1 (SW)
- new net: R76.2, R77.1, U20.1 (FB)
- new net: D10.1 (K), Q9.1 (G), R75.1
- new net: D12.1 (K), L2.2
- new net: C43.1, L1.1, U20.5 (SW)
- new net: C43.2, U20.6 (BST)
- new net +12V: C41.1, C42.2, C48.1, D11.2 (A2), Q9.3 (D), U20.2 (EN), U20.3 (IN), U22.4 (EN), U22.5 (VIN)
- new net +3.3V: C47.1, FB1.1, U21.5 (OUT)
- new net +3.3VA: C50.1, C51.1, FB1.2
- new net +30V: C49.1, D12.2 (A), R78.1
- new net +5V: C44.2, C45.1, L1.2, R76.1, U21.1 (IN), U21.3 (EN)
- new net GND: C41.2, C42.1, C44.1, C45.2, C46.2, C47.2, C48.2, C49.2, D11.1 (A1), J4.2 (Pin_2), R75.2, R77.2, R79.2, R80.1, U20.4 (GND), U21.2 (GND), U22.2 (GND)
- new net GNDA: C50.2, C51.2, R80.2
- new net VIN_RAW: D10.2 (A), F1.2, Q9.2 (S)
Other:
- note added: "12V => 28V"
- note added: "12V => 5V"
- note added: "5V => 3.3V"
- note added: "AP63203's reference: 0.8V 10/62.3×5 = 0.803V"
- note added: "Analog rail"
- note added: "Grounds"
- note added: "Input protection chain"
- note added: "TPS61040's reference: 1.233V 1.233×(215+10)/10 = 27.7V"
