File: can.kicad_sch (KiCad schematic)
At the start: 0 parts

Commit message: can transceiver; power; mcu
Parts:
- added C38, C39: 100nF, symbol Device:C
- added C40: C, symbol Device:C
- added R73, R74: 60.4, symbol Device:R
- added U19: TJA1051T-3, Package_SO:SOIC-8_3.9x4.9mm_P1.27mm, symbol Interface_CAN_LIN:TJA1051T-3
Connections:
- new net: C40.1, R73.2, R74.2
- new net +3.3V: C39.1, U19.5 (VIO)
- new net +5V: C38.2, U19.3 (VCC)
- new net CANH: R73.1, U19.7 (CANH)
- new net CANL: R74.1, U19.6 (CANL)
- new net CAN_RX: U19.4 (RXD)
- new net CAN_TX: U19.1 (TXD)
- new net GND: C38.1, C39.2, C40.2, U19.2 (GND), U19.8 (S)
Other:
- note added: "CAN Termination DNP unless end of bus"
- note added: "Datasheet: https://www.nxp.com/docs/en/data-sheet/TJA1051.pdf CAN is differential sensing, so it rejects the common-mode noise a motor controller injects. Degrades to single-wire. Priority-based arbitration, so a fault frame wins the bus."
- note added: "S is tied to GND directly. HIGH selects Silent mode (receives but never transmits)"
- note added: "bus side"
- note added: "logic side"

Commit message: Add presentation (slides, PDF, pptx) and latest schematic edits
Parts:
- C40: value C -> 4.7nF
Changed lines of the file:
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@@
 			)
 		)
-		(property "Value" "C"
+		(property "Value" "4.7nF"
 			(at 172.72 78.74 90)
 			(show_name no)
