File: feb-bms.kicad_sch (KiCad schematic)
At the start: 7 parts, among them J1 cell_taps, J2 temp_sensor, J3 CAN, J4 POWER_IN, J5 SDC, J6 Conn_ARM_JTAG_SWD_10, J7 AMS

Commit message: can transceiver; power; mcu
Parts:
- removed J4: POWER_IN, symbol Connector:Conn_01x02_Socket
- added D9: PESD1CAN, symbol Device:D_TVS_Dual_ACA
Connections:
- net GND: now also D9.2 (common)
- net CANH renamed can/CANH
- net can/CANH: now also D9.1 (A1)
- net CANL renamed can/CANL
- net can/CANL: now also D9.3 (A2)
Other:
- sheet balance ports: added BAL_EN[1..6], CELL[1..7]; removed none
- sheet can ports: added CAN, CANH, CANL; removed none
- sheet frontend ports: added CELL[1..7], FE_CTL, VCELL; removed none
- sheet mcu ports: added BAL_EN[1..6], CAN, FAULT_N, FE_CTL, SWD, TEMP[1..6], VCELL, VREF_MON, WDT_KICK; removed none
- sheet temp ports: added TEMP[1..6], TEMP_HOT, TSENSE[1..6]; removed none
- moved on the sheet: J3

Commit message: Add presentation (slides, PDF, pptx) and latest schematic edits
Other:
- added sheet differential-sensing (differential-sensing.kicad_sch)
Changed lines of the file:
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@@
+	)
+	(sheet
+		(at 33.655 80.01)
+		(size 21.59 13.335)
+		(exclude_from_sim no)
+		(in_bom yes)
+		(on_board yes)
+		(dnp no)
+		(fields_autoplaced yes)
+		(stroke
+			(width 0.1524)
+			(type solid)
+		)
+		(fill
+			(color 0 0 0 0)
+		)
+		(property "Sheetname" "differential-sensing"
+			(at 33.655 79.2984 0)
+			(show_name no)
+			(do_not_autoplace no)
+			(effects
+				(font
+					(size 1.27 1.27)
+				)
+				(justify left bottom)
+			)
+		)
+		(property "Sheetfile" "differential-sensing.kicad_sch"
+			(at 33.655 93.9296 0)
+			(show_name no)
+			(do_not_autoplace no)
+			(effects
+				(font
+					(size 1.27 1.27)
+				)
+				(justify left top)
+			)
+		)
+		(instances
+			(project "feb-bms"
+				(path "/6d76ad74-633b-4854-84fa-dd9a481927d0"
+					(page "9")
+				)
+			)
+		)
 	)
 	(sheet
