File: mcu.kicad_sch (KiCad schematic)
At the start: 0 parts

Commit message: can transceiver; power; mcu
Parts:
- added C25, C28, C30, C32, C33, C35, C37: 100nF, symbol Device:C
- added C26, C27, C29, C31: 10uF, symbol Device:C
- added C34: 1uF, symbol Device:C
- added C36: 2.2uF, symbol Device:C
- added R71, R72: 10k, symbol Device:R
- added U18: STM32F446RETx, Package_QFP:LQFP-64_10x10mm_P0.5mm, symbol MCU_ST_STM32F4:STM32F446RETx
Connections:
- new net: R71.1, U18.60 (BOOT0)
- new net: R72.1, U18.7 (NRST)
- new net: C33.2, U18.1 (VBAT)
- new net: C36.1, U18.30 (VCAP_1)
- new net: C34.2, C35.1
- new net +3.3V: C25.2, C26.2, C27.2, C28.2, C29.2, C30.2, C31.2, C32.2, C33.1, C37.1, R72.2, U18.19 (VDD), U18.32 (VDD), U18.48 (VDD), U18.64 (VDD)
- new net +3.3VA: C34.1, U18.13 (VDDA)
- new net BAL_EN1: U18.56 (PB4)
- new net BAL_EN2: U18.57 (PB5)
- new net BAL_EN3: U18.58 (PB6)
- new net BAL_EN4: U18.59 (PB7)
- new net BAL_EN5: U18.33 (PB12)
- new net BAL_EN6: U18.34 (PB13)
- new net CAN_RX: U18.61 (PB8)
- new net CAN_TX: U18.62 (PB9)
- new net FAULT_N: U18.41 (PA8)
- new net GND: C25.1, C26.1, C27.1, C28.1, C29.1, C30.1, C31.1, C32.1, C36.2, C37.2, R71.2, U18.18 (VSS), U18.31 (VSS), U18.47 (VSS), U18.63 (VSS)
- new net GNDA: C35.2, U18.12 (VSSA)
- new net MUX_A0: U18.37 (PC6)
- new net MUX_A1: U18.38 (PC7)
- new net MUX_A2: U18.39 (PC8)
- new net MUX_EN: U18.40 (PC9)
- new net SWCLK: U18.49 (PA14)
- new net SWDIO: U18.46 (PA13)
- new net SWO: U18.55 (PB3)
- new net TEMP1: U18.15 (PA1)
- new net TEMP2: U18.16 (PA2)
- new net TEMP3: U18.17 (PA3)
- new net TEMP4: U18.20 (PA4)
- new net TEMP5: U18.21 (PA5)
- new net TEMP6: U18.22 (PA6)
- new net VCELL: U18.14 (PA0)
- new net VREF_MON: U18.23 (PA7)
- new net WDT_KICK: U18.51 (PC10)

Commit message: Add presentation (slides, PDF, pptx) and latest schematic edits
Connections:
- no-connect marks 0 -> 25
Changed lines of the file:
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@@
 		(color 0 0 0 0)
+	)
+	(no_connect
+		(at 156.21 118.11)
+	)
+	(no_connect
+		(at 156.21 120.65)
+	)
+	(no_connect
+		(at 115.57 110.49)
+	)
+	(no_connect
+		(at 115.57 87.63)
+	)
+	(no_connect
+		(at 115.57 107.95)
+	)
+	(no_connect
+		(at 115.57 133.35)
+	)
+	(no_connect
+		(at 115.57 130.81)
+	)
+	(no_connect
+		(at 156.21 100.33)
+	)
+	(no_connect
+		(at 115.57 100.33)
+	)
+	(no_connect
+		(at 115.57 125.73)
+	)
+	(no_connect
+		(at 156.21 153.67)
+	)
+	(no_connect
+		(at 156.21 102.87)
+	)
+	(no_connect
+		(at 156.21 143.51)
+	)
+	(no_connect
+		(at 115.57 102.87)
+	)
+	(no_connect
+		(at 156.21 151.13)
+	)
+	(no_connect
+		(at 115.57 97.79)
+	)
+	(no_connect
+		(at 115.57 92.71)
+	)
+	(no_connect
+		(at 156.21 113.03)
+	)
+	(no_connect
+		(at 115.57 135.89)
+	)
+	(no_connect
+		(at 156.21 97.79)
+	)
+	(no_connect
+		(at 156.21 105.41)
+	)
+	(no_connect
+		(at 115.57 105.41)
+	)
+	(no_connect
+		(at 115.57 128.27)
+	)
+	(no_connect
+		(at 115.57 85.09)
+	)
+	(no_connect
+		(at 156.21 123.19)
 	)
 	(bus_entry
